File: layout/cam_board/cam_board.kicad_pcb (KiCad board)
At the start: 2 copper layers, 12 parts, among them U1 STM32F401CCUx

Commit message: Update layout and schematic
Parts:
- added C12: 100nF, Capacitor_SMD:C_0603_1608Metric_Pad1.08x0.95mm_HandSolder, F.Cu at (105.2, 93.1)
- added C13: 100nF, Capacitor_SMD:C_0603_1608Metric_Pad1.08x0.95mm_HandSolder, F.Cu at (105.2, 95.8)
- added C14: 100nF, Capacitor_SMD:C_0603_1608Metric_Pad1.08x0.95mm_HandSolder, F.Cu at (139.8, 70.9)
- added C15: 10uF, Capacitor_SMD:C_0603_1608Metric_Pad1.08x0.95mm_HandSolder, F.Cu at (139.8, 73.4)
- added C16: 10uF, Capacitor_SMD:C_0603_1608Metric_Pad1.08x0.95mm_HandSolder, F.Cu at (139.8, 75.9)
- added C17: 10uF, Capacitor_SMD:C_0603_1608Metric_Pad1.08x0.95mm_HandSolder, F.Cu at (139.8, 78.4)
- added C18: 100nF, Capacitor_SMD:C_0603_1608Metric_Pad1.08x0.95mm_HandSolder, F.Cu at (159.2, 94.9)
- added C19: 100nF, Capacitor_SMD:C_0603_1608Metric_Pad1.08x0.95mm_HandSolder, F.Cu at (137.6, 104.8)
- added C20: 4u7F, Capacitor_SMD:C_0603_1608Metric_Pad1.08x0.95mm_HandSolder, F.Cu at (161.7, 82.2)
- added D1: USER_LED, LED_SMD:LED_0603_1608Metric_Pad1.05x0.95mm_HandSolder, F.Cu at (144.2, 84.0)
- added D2: D_Zener, Diode_SMD:D_0201_0603Metric_Pad0.64x0.40mm_HandSolder, F.Cu at (143.6, 88.8)
- added D3: PWRLED, LED_SMD:LED_0603_1608Metric_Pad1.05x0.95mm_HandSolder, F.Cu at (144.2, 86.6)
- added D4: CHARGINGLED, LED_SMD:LED_0603_1608Metric_Pad1.05x0.95mm_HandSolder, F.Cu at (166.1, 87.0)
- added R1: 10k, Resistor_SMD:R_0603_1608Metric_Pad0.98x0.95mm_HandSolder, F.Cu at (101.5, 93.7)
- added R2: 10k, Resistor_SMD:R_0603_1608Metric_Pad0.98x0.95mm_HandSolder, F.Cu at (101.5, 97.4)
- added R3: 10k, Resistor_SMD:R_0603_1608Metric_Pad0.98x0.95mm_HandSolder, F.Cu at (139.8, 80.9)
- added R4: 5k1, Resistor_SMD:R_0603_1608Metric_Pad0.98x0.95mm_HandSolder, F.Cu at (139.8, 83.4)
- added R5: 5k1, Resistor_SMD:R_0603_1608Metric_Pad0.98x0.95mm_HandSolder, F.Cu at (139.8, 85.9)
- added R6: 10k, Resistor_SMD:R_0603_1608Metric_Pad0.98x0.95mm_HandSolder, F.Cu at (139.8, 88.4)
- added R7: 10k, Resistor_SMD:R_0603_1608Metric_Pad0.98x0.95mm_HandSolder, F.Cu at (159.2, 97.4)
- added R8: 2k, Resistor_SMD:R_0603_1608Metric_Pad0.98x0.95mm_HandSolder, F.Cu at (161.7, 84.7)
- added R9: 10k, Resistor_SMD:R_0603_1608Metric_Pad0.98x0.95mm_HandSolder, F.Cu at (161.7, 87.2)
- added SW1: SW_MEC_5E, Button_Switch_SMD:SW_MEC_5GSH9, F.Cu at (105.3, 83.5)
- added SW2: SW_MEC_5E, Button_Switch_SMD:SW_MEC_5GSH9, F.Cu at (116.9, 83.5)
- added SW3: SW_MEC_5E, Button_Switch_SMD:SW_MEC_5GSH9, F.Cu at (151.2, 102.0)
- added U2: USBLC6-2SC6, Package_TO_SOT_SMD:SOT-23-6_Handsoldering, F.Cu at (144.9, 80.4)
- added U3: LD1117S33TR_SOT223, Package_TO_SOT_SMD:SOT-223-3_TabPin2, F.Cu at (146.9, 73.8)
- added U4: MCP73831-2-OT, Package_TO_SOT_SMD:SOT-23-5_HandSoldering, F.Cu at (166.8, 83.4)
- C1, C10, C11, C2, C3, C4, C5, C6, C7, C8, C9: footprint Capacitor_SMD:C_0504_1310Metric_Pad0.83x1.28mm_HandSolder -> Capacitor_SMD:C_0603_1608Metric_Pad1.08x0.95mm_HandSolder
Connections:
- net Net-(U1-VCAP1) renamed VCAP1
- C2 pad 2: +3V3 -> VBAT
- C3 pad 2: +3V3 -> VBAT
- C4 pad 2: +3V3 -> VBAT
- C5 pad 2: +3V3 -> VBAT
- C6 pad 2: +3V3 -> VBAT
- C7 pad 2: +3V3 -> VBAT
- U1 pad 1: unconnected-(U1-VBAT-Pad1) -> VBAT
- U1 pad 24: +3V3 -> VBAT
- U1 pad 32: unconnected-(U1-PA11-Pad32) -> D-
- U1 pad 33: unconnected-(U1-PA12-Pad33) -> D+
- U1 pad 36: +3V3 -> VBAT
- U1 pad 48: +3V3 -> VBAT
- U1 pad 9: +3V3 -> VBAT

Commit message: Update layout and schematic
Parts:
- removed D2: D_Zener, Diode_SMD:D_0201_0603Metric_Pad0.64x0.40mm_HandSolder
- removed D3: PWRLED, LED_SMD:LED_0603_1608Metric_Pad1.05x0.95mm_HandSolder
- removed D4: CHARGINGLED, LED_SMD:LED_0603_1608Metric_Pad1.05x0.95mm_HandSolder
- removed U4: MCP73831-2-OT, Package_TO_SOT_SMD:SOT-23-5_HandSoldering
- added C21: 4u7F, Capacitor_SMD:C_0603_1608Metric_Pad1.08x0.95mm_HandSolder, F.Cu at (133.4, 86.0)
- added C22: 4u7F, Capacitor_SMD:C_0603_1608Metric_Pad1.08x0.95mm_HandSolder, F.Cu at (137.8, 71.0)
- added C23: 10nF, Capacitor_SMD:C_0603_1608Metric_Pad1.08x0.95mm_HandSolder, F.Cu at (137.8, 73.5)
- added D5: D_Schottky, Diode_SMD:D_0603_1608Metric_Pad1.05x0.95mm_HandSolder, F.Cu at (157.5, 82.9)
- added Q1: BSS138, Package_TO_SOT_SMD:SOT-23_Handsoldering, F.Cu at (160.7, 89.8)
- added R10: 2k, Resistor_SMD:R_0603_1608Metric_Pad0.98x0.95mm_HandSolder, F.Cu at (142.1, 81.0)
- added R11: 2k, Resistor_SMD:R_0603_1608Metric_Pad0.98x0.95mm_HandSolder, F.Cu at (142.1, 83.5)
- added R12: 100k, Resistor_SMD:R_0603_1608Metric_Pad0.98x0.95mm_HandSolder, F.Cu at (142.1, 86.0)
- added R13: 10k, Resistor_SMD:R_0603_1608Metric_Pad0.98x0.95mm_HandSolder, F.Cu at (146.4, 71.0)
- added R14: 10k, Resistor_SMD:R_0603_1608Metric_Pad0.98x0.95mm_HandSolder, F.Cu at (146.4, 73.5)
- added R15: 10k, Resistor_SMD:R_0603_1608Metric_Pad0.98x0.95mm_HandSolder, F.Cu at (146.4, 76.0)
- added R16: 10k, Resistor_SMD:R_0603_1608Metric_Pad0.98x0.95mm_HandSolder, F.Cu at (146.4, 78.5)
- added R17: 100k, Resistor_SMD:R_0603_1608Metric_Pad0.98x0.95mm_HandSolder, F.Cu at (146.4, 81.0)
- added R18: 100k, Resistor_SMD:R_0603_1608Metric_Pad0.98x0.95mm_HandSolder, F.Cu at (146.4, 83.5)
- added U5: MCP73871-1AA, Package_DFN_QFN:QFN-20-1EP_4x4mm_P0.5mm_EP2.5x2.5mm_ThermalVias, F.Cu at (152.1, 82.2)
- R8: value 2k -> 10k
- U3: value LD1117S33TR_SOT223 -> MCP1700x-330xxTT; footprint Package_TO_SOT_SMD:SOT-223-3_TabPin2 -> Package_TO_SOT_SMD:SOT-23_Handsoldering
- moved R2 40.9 mm to (137.8, 78.5)
- moved R1 40.4 mm to (137.8, 76.0)
- moved C18 30.6 mm to (133.4, 78.5)
- moved R7 29.4 mm to (142.1, 73.5)
- moved U1 28.9 mm to (153.7, 74.4)
- moved C20 28.4 mm to (133.4, 83.5)
- moved C13 26.8 mm to (129.1, 83.5)
- moved C12 26.8 mm to (129.1, 81.0)
- moved SW2 26.1 mm to (140.0, 95.6)
- moved SW1 26.1 mm to (128.3, 95.6)
- moved U3 25.0 mm to (160.7, 94.6)
- moved U2 24.5 mm to (160.4, 99.3)
- moved C19 24.1 mm to (133.4, 81.0)
- moved R8 21.5 mm to (142.1, 76.0)
- moved R9 21.5 mm to (142.1, 78.5)
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Connections:
- C14 pad 2: +5V -> USB+5V
- C15 pad 2: +5V -> USB+5V
- C16 pad 2: +5V -> VOUT
- C20 pad 2: +BATT -> Net-(J3-Pin_2)
- R6 pad 1: Net-(D3-A) -> VOUT
- R6 pad 2: VBAT -> Net-(U5-VPCC)
- R8 pad 1: Net-(U4-PROG) -> VOUT
- R8 pad 2: GND -> Net-(U5-CE)
- R9 pad 1: +5V -> VOUT
- U1 pad 16: unconnected-(U1-PA6-Pad16) -> BATTLVL
- U1 pad 26: unconnected-(U1-PB13-Pad26) -> BATTFULL
- U1 pad 27: unconnected-(U1-PB14-Pad27) -> BATTCHARGE
- U1 pad 28: unconnected-(U1-PB15-Pad28) -> EXT_POWER
- U2 pad 5: +5V -> USB+5V
- U3 pad 3: +5V -> VOUT

Commit message: First full schematic
Parts:
- removed U3: MCP1700x-330xxTT, Package_TO_SOT_SMD:SOT-23_Handsoldering
- added A1: MLX90640ESF-BAA-000-TU, A_Custom:TO292P930H600-4-MLX, F.Cu at (143.9, 100.4)
- added C24: 100nF, Capacitor_SMD:C_0603_1608Metric_Pad1.08x0.95mm_HandSolder, F.Cu at (123.1, 92.8)
- added C25: 10u, Capacitor_SMD:C_0603_1608Metric_Pad1.08x0.95mm_HandSolder, F.Cu at (123.1, 95.3)
- added D2: D_Schottky, Diode_SMD:D_0603_1608Metric_Pad1.05x0.95mm_HandSolder, F.Cu at (136.2, 87.9)
- added D3: D_Schottky, Diode_SMD:D_0603_1608Metric_Pad1.05x0.95mm_HandSolder, F.Cu at (136.2, 90.5)
- added D4: POWER_LED, LED_SMD:LED_0603_1608Metric_Pad1.05x0.95mm_HandSolder, F.Cu at (136.2, 93.0)
- added J1: Debug, Connector_PinHeader_1.27mm:PinHeader_1x06_P1.27mm_Vertical, F.Cu at (151.4, 96.1)
- added J2: USB Connector, Connector_USB:USB_C_Receptacle_HRO_TYPE-C-31-M-12, F.Cu at (144.2, 89.8)
- added J3: BATT_CONNECTOR, Connector_JST:JST_PH_B2B-PH-K_1x02_P2.00mm_Vertical, F.Cu at (150.2, 79.4)
- added J4: LCD conn, Connector_PinHeader_1.27mm:PinHeader_1x08_P1.27mm_Vertical, F.Cu at (136.1, 98.6)
- added J5: Stick conn, Connector_PinHeader_1.27mm:PinHeader_1x05_P1.27mm_Vertical, F.Cu at (155.6, 96.1)
- added JP1: BypassBattery, Jumper:SolderJumper-3_P1.3mm_Open_RoundedPad1.0x1.5mm_NumberLabels, F.Cu at (152.9, 92.0)
- added R19: 1k, Resistor_SMD:R_0603_1608Metric_Pad0.98x0.95mm_HandSolder, F.Cu at (131.8, 92.8)
- added R21: 1k, Resistor_SMD:R_0603_1608Metric_Pad0.98x0.95mm_HandSolder, F.Cu at (131.8, 95.3)
- added R22: 1k, Resistor_SMD:R_0603_1608Metric_Pad0.98x0.95mm_HandSolder, F.Cu at (131.8, 97.8)
- added SW4: Sys On/Off, Button_Switch_SMD:SW_DIP_SPSTx01_Slide_6.7x4.1mm_W6.73mm_P2.54mm_LowProfile_JPin, F.Cu at (143.6, 108.8)
- added U4: AP2112K-3.3, Package_TO_SOT_SMD:SOT-23-5_HandSoldering, F.Cu at (127.5, 111.5)
- added Y1: ECS-80-18-23B-JTN-TR, A_Custom:XTAL_ECS-80-18-23B-JTN-TR, F.Cu at (153.3, 106.8)
- added Y2: SC32S-7PF20PPM, A_Custom:XTAL_CM8V-T1A-32.768KHZ-6PF-20PPM-TA-QC, F.Cu at (151.2, 111.4)
- R3: value 10k -> 1k
- moved Q1 50.2 mm to (115.5, 111.6)
- moved U2 40.6 mm to (121.6, 111.5)
- moved R13 37.0 mm to (127.5, 102.8)
- moved R14 37.0 mm to (127.5, 105.3)
- moved R15 37.0 mm to (127.5, 107.8)
- moved C10 35.0 mm to (114.4, 107.8)
- moved C8 35.0 mm to (114.4, 102.8)
- moved C9 35.0 mm to (114.4, 105.3)
- moved C17 28.3 mm to (118.8, 100.3)
- moved C15 28.3 mm to (118.8, 95.3)
- moved C16 28.3 mm to (118.8, 97.8)
- moved C18 28.3 mm to (118.8, 102.8)
- moved C19 28.3 mm to (118.8, 105.3)
- moved C20 28.3 mm to (118.8, 107.8)
- moved R1 26.2 mm to (123.1, 97.8)
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Connections:
- net USER_BUTTON renamed USRBUTTON
- C16 pad 1: GND -> VOUT
- C16 pad 2: VOUT -> GND
- C21 pad 2: USB+5V -> Net-(JP1-B)
- C22 pad 2: Net-(SW4A-B) -> VOUT
- R8 pad 1: VOUT -> Net-(U5-CE)
- R8 pad 2: Net-(U5-CE) -> VOUT
- U1 pad 25: unconnected-(U1-PB12-Pad25) -> BATTLVL_READ
- U1 pad 39: unconnected-(U1-PB3-Pad39) -> SWO
- U5 pad 1: Net-(SW4A-B) -> VOUT
- U5 pad 18: USB+5V -> Net-(JP1-B)
- U5 pad 19: USB+5V -> Net-(JP1-B)
- U5 pad 20: Net-(SW4A-B) -> VOUT

Commit message: Update layout and schematic
Parts:
- removed C6: 1uF, Capacitor_SMD:C_0603_1608Metric_Pad1.08x0.95mm_HandSolder
- removed C7: 100nF, Capacitor_SMD:C_0603_1608Metric_Pad1.08x0.95mm_HandSolder
- added C26: 100nF, Capacitor_SMD:C_0402_1005Metric_Pad0.74x0.62mm_HandSolder, F.Cu at (86.4, 62.9)
- added C27: 1uF, Capacitor_SMD:C_0402_1005Metric_Pad0.74x0.62mm_HandSolder, F.Cu at (86.4, 61.7)
- added D6: CHARGING, LED_SMD:LED_0603_1608Metric_Pad1.05x0.95mm_HandSolder, F.Cu at (116.8, 71.4)
- added JP2: Prog1, Jumper:SolderJumper-3_P1.3mm_Open_RoundedPad1.0x1.5mm_NumberLabels, F.Cu at (119.0, 56.5)
- added JP3: Prog2, Jumper:SolderJumper-3_P1.3mm_Open_RoundedPad1.0x1.5mm_NumberLabels, F.Cu at (108.6, 63.4)
- added JP4: Prog1, Jumper:SolderJumper-3_P1.3mm_Open_RoundedPad1.0x1.5mm_NumberLabels, F.Cu at (119.0, 63.2)
- added R20: 110k, Resistor_SMD:R_0603_1608Metric_Pad0.98x0.95mm_HandSolder, F.Cu at (109.3, 57.8)
- C1, C10, C11, C19, C2, C3, C4, C5, C8, C9: footprint Capacitor_SMD:C_0603_1608Metric_Pad1.08x0.95mm_HandSolder -> Capacitor_SMD:C_0402_1005Metric_Pad0.74x0.62mm_HandSolder
- R10: value 2k -> 10k
- R12: value 100k -> 20k
- R14: value 10k -> 1k
- R18: value 100k -> 220k
- R6: value 10k -> 330K
- R9: value 10k -> 100k
- SW1: value SW_MEC_5E -> BOOT0; footprint Button_Switch_SMD:SW_MEC_5GSH9 -> Button_Switch_SMD:SW_DIP_SPSTx01_Slide_9.78x4.72mm_W8.61mm_P2.54mm
- SW2: value SW_MEC_5E -> NRST; footprint Button_Switch_SMD:SW_MEC_5GSH9 -> Button_Switch_SMD:SW_DIP_SPSTx01_Slide_9.78x4.72mm_W8.61mm_P2.54mm
- SW3: value SW_MEC_5E -> USER; footprint Button_Switch_SMD:SW_MEC_5GSH9 -> A_Custom:SW_1825910-6-4
- SW4: value Sys On/Off -> ON/OFF; footprint Button_Switch_SMD:SW_DIP_SPSTx01_Slide_6.7x4.1mm_W6.73mm_P2.54mm_LowProfile_JPin -> Button_Switch_SMD:SW_DIP_SPSTx01_Slide_9.78x4.72mm_W8.61mm_P2.54mm
- moved A1 90.1 mm to (96.2, 23.9)
- moved U2 89.9 mm to (116.0, 21.9)
- moved Y2 82.9 mm to (86.5, 59.6), turned to 90 degrees
- moved Y1 79.9 mm to (84.2, 66.7)
- moved J1 79.0 mm to (105.8, 31.5), turned to 90 degrees
- moved R22 79.0 mm to (103.3, 24.1)
- moved R21 79.0 mm to (103.3, 21.6)
- moved C24 76.9 mm to (88.9, 23.9)
- moved C25 76.9 mm to (88.9, 26.4)
- moved R4 74.1 mm to (124.8, 31.2)
- moved R5 74.1 mm to (124.8, 33.7)
- moved SW3 70.9 mm to (71.2, 65.9), turned to 90 degrees
- moved SW2 66.2 mm to (67.9, 52.1)
- moved R3 65.5 mm to (83.3, 50.8), turned to 90 degrees
- moved D1 65.4 mm to (82.6, 47.8)
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Connections:
- net VCAP1 renamed Net-(U1-VCAP1)
- A1 pad 2: VBAT -> +3V3
- C17 pad 2: VBAT -> +3V3
- C19 pad 2: VBAT -> +3V3
- C2 pad 2: VBAT -> +3V3
- C24 pad 2: VBAT -> +3V3
- C25 pad 2: VBAT -> +3V3
- C3 pad 2: VBAT -> +3V3
- C4 pad 2: VBAT -> +3V3
- C5 pad 2: VBAT -> +3V3
- D2 pad 1: Net-(D2-K) -> VIN
- D3 pad 1: Net-(D2-K) -> VIN
- J4 pad 8: VBAT -> +3V3
- J5 pad 5: VBAT -> +3V3
- JP1 pad 2: Net-(D2-K) -> VIN
- R1 pad 1: VBAT -> +3V3
- R10 pad 1: VOUT -> Net-(JP2-A)
- R10 pad 2: Net-(U5-PROG2) -> VIN
- R11 pad 1: VOUT -> Net-(JP2-B)
- R11 pad 2: Net-(U5-PROG1) -> VIN
- R12 pad 1: GND -> Net-(JP4-B)
- R12 pad 2: Net-(U5-PROG3) -> VIN
- R14 pad 1: BATTCHARGE -> BATTCHARGING
- R14 pad 2: VBAT -> Net-(D6-A)
- R15 pad 2: VBAT -> VIN
- R16 pad 2: VBAT -> VIN
- R17 pad 2: VOUT -> Net-(J3-Pin_2)
- R19 pad 1: VBAT -> +3V3
- R21 pad 1: VBAT -> +3V3
- R22 pad 1: VBAT -> +3V3
- R6 pad 1: VOUT -> Net-(U5-VPCC)
- R6 pad 2: Net-(U5-VPCC) -> VIN
- R8 pad 1: Net-(U5-CE) -> VIN
- R8 pad 2: VOUT -> BATTCHARGE
- R9 pad 1: VOUT -> Net-(JP4-A)
- R9 pad 2: Net-(U5-SEL) -> VIN
- SW1 pad 1: VBAT -> +3V3
- SW1 pad 2: VBAT -> BOOT0
- SW2 pad 2: GND -> NRST
- SW3 pad 1: VBAT -> +3V3
- SW3 pad 2: VBAT -> +3V3
- SW4 pad 1: Net-(SW4-B) -> VOUT
- SW4 pad 2: VOUT -> GND
- U1 pad 1: VBAT -> +3V3
- U1 pad 21: unconnected-(U1-PB10-Pad21) -> BATTCHARGE
- U1 pad 24: VBAT -> +3V3
- U1 pad 27: BATTCHARGE -> BATTCHARGING
- U1 pad 36: VBAT -> +3V3
- U1 pad 48: VBAT -> +3V3
- U1 pad 9: VBAT -> +3V3
- U4 pad 3: Net-(SW4-B) -> GND
- U4 pad 5: VBAT -> +3V3
- U5 pad 12: Net-(U5-PROG3) -> Net-(JP4-C)
- U5 pad 13: Net-(U5-PROG1) -> Net-(JP2-C)
- U5 pad 17: Net-(U5-CE) -> BATTCHARGE
- U5 pad 3: Net-(U5-SEL) -> GND
- U5 pad 4: Net-(U5-PROG2) -> Net-(JP3-C)
- U5 pad 8: BATTCHARGE -> BATTCHARGING

Commit message: Update layout and schematic
Parts:
- C23: footprint Capacitor_SMD:C_0603_1608Metric_Pad1.08x0.95mm_HandSolder -> Capacitor_SMD:C_0402_1005Metric_Pad0.74x0.62mm_HandSolder
- moved U2 47.5 mm to (108.8, 68.8), turned to 180 degrees
- moved SW4 40.6 mm to (97.8, 48.6), turned to 180 degrees
- moved R4 40.3 mm to (116.5, 70.6)
- moved C15 39.8 mm to (109.5, 66.0), turned to 180 degrees
- moved C14 36.6 mm to (115.6, 62.8)
- moved J2 36.1 mm to (123.6, 68.6)
- moved J1 35.3 mm to (126.2, 60.4), turned to 180 degrees
- moved R5 34.1 mm to (116.5, 66.8)
- moved R22 25.1 mm to (89.0, 44.8)
- moved C20 24.9 mm to (120.0, 34.3)
- moved C17 24.3 mm to (110.1, 58.0)
- moved D2 24.2 mm to (120.3, 60.0)
- moved D3 23.7 mm to (120.2, 57.4), turned to 0 degrees
- moved J3 23.5 mm to (124.3, 38.0), turned to 90 degrees
- moved R17 22.9 mm to (118.8, 36.9), turned to 90 degrees
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Connections:
- C17 pad 1: GND -> +3V3
- C17 pad 2: +3V3 -> GND
- J1 pad 1: SWO -> GND
- J1 pad 2: NRST -> SWD+5V
- J1 pad 3: SWDIO -> SWCLK
- J1 pad 4: GND -> SWDIO
- J1 pad 5: SWCLK -> SWO
- J1 pad 6: SWD+5V -> NRST
- U1 pad 10: USRBUTTON -> unconnected-(U1-PA0-Pad10)
- U1 pad 11: unconnected-(U1-PA1-Pad11) -> USER_LED
- U1 pad 2: USER_LED -> unconnected-(U1-PC13-Pad2)
- U1 pad 21: BATTCHARGE -> BL
- U1 pad 30: unconnected-(U1-PA9-Pad30) -> BATTCHARGE
- U1 pad 41: BL -> unconnected-(U1-PB5-Pad41)
- U1 pad 46: unconnected-(U1-PB9-Pad46) -> USRBUTTON
Routing:
- net GND: track 0.00 -> 100.6 mm, vias 0 -> 52
- net NRST: track 0.00 -> 71.1 mm, vias 0 -> 2
- net BATTLVL: track 0.00 -> 64.2 mm, vias 0 -> 4
- net +3V3: track 0.00 -> 53.3 mm, vias 0 -> 15
- net VOUT: track 0.00 -> 50.9 mm
- net BATTCHARGE: track 0.00 -> 44.6 mm, vias 0 -> 2
- net BATTCHARGING: track 0.00 -> 40.5 mm, vias 0 -> 2
- net BATTFULL: track 0.00 -> 38.0 mm, vias 0 -> 2
- net EXT_POWER: track 0.00 -> 34.4 mm, vias 0 -> 2
- net SCL: track 0.00 -> 33.4 mm, vias 0 -> 1
- net SWO: track 0.00 -> 30.9 mm, vias 0 -> 1
- net SWDIO: track 0.00 -> 29.8 mm, vias 0 -> 1
- net BATTLVL_READ: track 0.00 -> 29.6 mm, vias 0 -> 4
- net USRBUTTON: track 0.00 -> 28.7 mm
- net SWCLK: track 0.00 -> 28.1 mm, vias 0 -> 1
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- added copper zone on In2.Cu, net +3V3
- added copper zone on B.Cu, net GND
- added copper zone on F.Cu, net GND
- added copper zone on In1.Cu, net GND
- added copper zone on In2.Cu, net VIN
Other:
- board outline added: 57.2 x 44.3 mm
- copper layers 2 -> 4

Commit message: Update layout and schematic
Parts:
- removed JP1: BypassBattery, Jumper:SolderJumper-3_P1.3mm_Open_RoundedPad1.0x1.5mm_NumberLabels
- moved R6 2.93 mm to (105.8, 40.2), turned to 180 degrees
- moved R20 2.11 mm to (105.8, 38.5)
- moved C22 0.92 mm to (108.8, 37.6)
- moved C10 0.75 mm to (87.6, 59.7)
- moved C11 0.75 mm to (87.6, 58.1)
- moved Y2 0.75 mm to (89.8, 58.8)
- moved C21 0.05 mm to (111.3, 38.0)
Connections:
- C21 pad 2: Net-(JP1-B) -> Net-(D2-K)
- D2 pad 1: VIN -> Net-(D2-K)
- D3 pad 1: VIN -> Net-(D2-K)
- U5 pad 18: Net-(JP1-B) -> Net-(D2-K)
- U5 pad 19: Net-(JP1-B) -> Net-(D2-K)
Routing:
- net Net-(D2-K): track 0.00 -> 51.8 mm
- net GND: track 100.6 -> 114.6 mm, vias 52 -> 54
- net VOUT: track 50.9 -> 40.3 mm, vias 0 -> 2
- net Net-(D5-A): track 6.88 -> 14.1 mm
- net VIN: track 20.1 -> 13.4 mm, vias 10 -> 9
- net Net-(JP1-B): track 3.74 -> 0.00 mm
- net +3V3: track 53.3 -> 56.5 mm, vias 15 -> 17
- net BATTLVL_READ: track 29.6 -> 32.3 mm
- net Net-(U5-VPCC): track 7.38 -> 5.48 mm
- net OSC32_OUT: track 4.09 -> 4.84 mm
- net OSC32_IN: track 5.05 -> 5.65 mm

Commit message: Update layout and schematic
Parts:
- moved SW4 2.36 mm to (95.4, 48.6)
- moved R21 1.55 mm to (97.5, 43.6), turned to -90 degrees
- moved D1 1.13 mm to (86.0, 69.1)
- moved C8 0.55 mm to (82.1, 63.2)
- moved C9 0.55 mm to (84.4, 59.9)
- moved Y1 0.55 mm to (86.2, 62.6)
Routing:
- net VOUT: track 40.3 -> 43.6 mm
- net GND: track 114.6 -> 117.5 mm
- net SDA: track 21.7 -> 19.4 mm
- net OSC_IN: track 7.44 -> 8.59 mm
- net Net-(D1-A): track 3.07 -> 1.95 mm
- net OSC_OUT: track 10.6 -> 11.5 mm
- net NRST: track 71.1 -> 71.9 mm
- net +3V3: track 56.5 -> 57.2 mm
- net USER_LED: track 8.88 -> 9.51 mm
Other:
- board size 57.2 x 44.3 mm -> 57.2 x 45.3 mm

Commit message: Update layout and schematic
Parts:
- added M1: MountingHole_2.1mm, MountingHole:MountingHole_2.1mm, F.Cu at (80.8, 34.5)
- added M2: MountingHole_2.1mm, MountingHole:MountingHole_2.1mm, F.Cu at (115.0, 75.2)
- A1, C24, C25, R21, R22: moved to B.Cu
- moved R21 14.5 mm to (83.0, 43.3), turned to 0 degrees
- moved C24 11.6 mm to (96.6, 39.3), turned to 180 degrees
- moved C25 8.44 mm to (95.0, 36.8), turned to 180 degrees
- moved R22 4.15 mm to (92.8, 46.5), turned to 180 degrees
- moved A1 3.09 mm to (89.6, 40.9), turned to 0 degrees
- moved D4 2.53 mm to (110.4, 61.0)
- moved R19 2.53 mm to (106.7, 61.0)
- moved C16 2.30 mm to (105.1, 56.5)
- moved C17 2.30 mm to (110.6, 55.8)
- moved U4 2.30 mm to (108.3, 58.3)
- moved C14 0.92 mm to (116.4, 62.2)
- moved J2 0.38 mm to (124.0, 68.6)
- moved R6 0.30 mm to (105.6, 40.5)
- moved R20 0.30 mm to (105.6, 38.6)
- moved D3 0.15 mm to (120.3, 57.4)
Connections:
- C21 pad 2: Net-(D2-K) -> VIN
- D2 pad 1: Net-(D2-K) -> VIN
- D3 pad 1: Net-(D2-K) -> VIN
- U5 pad 18: Net-(D2-K) -> VIN
- U5 pad 19: Net-(D2-K) -> VIN
Routing:
- net VIN: track 13.4 -> 70.7 mm, vias 9 -> 13
- net Net-(D2-K): track 52.2 -> 0.00 mm
- net GND: track 117.5 -> 102.8 mm, vias 54 -> 50
- net SDA: track 19.4 -> 26.8 mm
- net BATTLVL: track 64.2 -> 58.6 mm, vias 4 -> 2
- net SCL: track 33.5 -> 29.2 mm
- net +3V3: track 57.2 -> 53.2 mm, vias 17 -> 16
- net BATTLVL_READ: track 32.3 -> 30.7 mm, vias 4 -> 2
- net Net-(U5-VPCC): track 5.48 -> 7.00 mm
- net Net-(J3-Pin_2): track 21.7 -> 20.4 mm
- net VOUT: track 43.6 -> 42.7 mm, vias 2 -> 0
- net USRBUTTON: track 28.7 -> 29.3 mm
- net USB+5V: track 22.8 -> 22.3 mm
Other:
- board size 57.2 x 45.3 mm -> 58 x 46 mm
- board text added: "+"
- board text added: "+3V3"
- board text added: "+5V"
- board text added: "-"
- board text added: "BATTERY"
- board text added: "BL"
- board text added: "BOOT0"
- board text added: "CHARGING"
- board text added: "CLK"
- board text added: "CS"
- board text added: "DC"
- board text added: "DIN"
- board text added: "DISPLAY"
- board text added: "GND"
- board text added: "IR-Camera Bottom Version A L.Kratzl"
- board text added: "IR-Camera Top Version A L.Kratzl"
- board text added: "IR-SENSOR (BACK SIDE)"
- board text added: "JOYSTICK"
- board text added: "NRST"
- board text added: "ON/OFF"
- board text added: "POWER"
- board text added: "RST"
- board text added: "SCL"
- board text added: "SDA"
- board text added: "SWCLK"
- board text added: "SWD"
- board text added: "SWDIO"
- board text added: "SWO"
- board text added: "USB USER"
- board text added: "USER"
- board text added: "X"
- board text added: "Y"
- board text added: "Z"
