File: layout/cam_board/cam_board.kicad_sch (KiCad schematic)
At the start: 74 parts, among them J1 Debug, J2 USB Connector, J3 BATT_CONNECTOR, J4 LCD conn, J5 Stick conn, Q1 BSS138, SW1 BOOT0, SW2 NRST, SW3 USER, SW4 ON/OFF, U1 STM32F401CCUx, U2 USBLC6-2SC6, U4 AP2112K-3.3, U5 MCP73871-1AA, Y1 ECS-80-18-23B-JTN-TR, Y2 SC32S-7PF20PPM

Commit message: Update layout and schematic
Parts:
- removed JP1: BypassBattery, Jumper:SolderJumper-3_P1.3mm_Open_RoundedPad1.0x1.5mm_NumberLabels, symbol Jumper:SolderJumper_3_Open
Connections:
- net VIN: now also C21.2, U5.18 (IN), U5.19 (IN)
Other:
- note added: "NTE Low -> Security active"
- note added: "THERM low -> no temperatur-check"
- note added: "VBAT_SENSE -> Measure Battery voltage"
- note removed: "NTE Low -> Sicherheitstimer aktiv"
- note removed: "THERM low -> kein temperatur-check"
- note removed: "VBAT_SENSE -> Misst die Batteriespannung"
Changed lines of the file:
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@@
 		)
 	)
-	(text "THERM low -> kein temperatur-check"
+	(text "THERM low -> no temperatur-check"
 		(exclude_from_sim no)
 		(at 191.262 94.996 0)
@@
 		)
 	)
-	(text "NTE Low -> Sicherheitstimer aktiv"
+	(text "NTE Low -> Security active"
 		(exclude_from_sim no)
 		(at 189.484 92.71 0)
@@
 		)
 	)
-	(text "VBAT_SENSE -> Misst die Batteriespannung"
+	(text "VBAT_SENSE -> Measure Battery voltage"
 		(exclude_from_sim no)
 		(at 193.548 97.536 0)
@@
 	)
 	(junction
-		(at 227.33 29.21)
-		(diameter 0)
-		(color 0 0 0 0)
-	)
-	(junction
 		(at 182.88 118.11)
 		(diameter 0)
@@
 	)
 	(junction
-		(at 238.76 33.02)
-		(diameter 0)
-		(color 0 0 0 0)
-	)
-	(junction
 		(at 74.93 30.48)
 		(diameter 0)
@@
 	)
 	(junction
+		(at 224.79 29.21)
+		(diameter 0)
+		(color 0 0 0 0)
+	)
+	(junction
 		(at 46.99 185.42)
 		(diameter 0)
@@
 	(wire
 		(pts
-			(xy 224.79 29.21) (xy 227.33 29.21)
+			(xy 224.79 29.21) (xy 237.49 29.21)
 		)
 		(stroke
@@
 	(wire
 		(pts
-			(xy 232.41 33.02) (xy 238.76 33.02)
-		)
-		(stroke
-			(width 0)
-			(type default)
-		)
-	)
-	(wire
-		(pts
 			(xy 220.98 81.28) (xy 220.98 83.82)
 		)
@@
 	(wire
 		(pts
-			(xy 222.25 33.02) (xy 220.98 33.02)
+			(xy 220.98 33.02) (xy 224.79 33.02)
 		)
 		(stroke
@@
 	(wire
 		(pts
+			(xy 224.79 27.94) (xy 224.79 29.21)
+		)
+		(stroke
+			(width 0)
+			(type default)
+		)
+	)
+	(wire
+		(pts
 			(xy 154.94 69.85) (xy 156.21 69.85)
 		)
@@
 	(wire
 		(pts
-			(xy 227.33 29.21) (xy 237.49 29.21)
-		)
-		(stroke
-			(width 0)
-			(type default)
-		)
-	)
-	(wire
-		(pts
 			(xy 85.09 140.97) (xy 83.82 140.97)
 		)
@@
 	(wire
 		(pts
-			(xy 224.79 27.94) (xy 224.79 29.21)
-		)
-		(stroke
-			(width 0)
-			(type default)
-		)
-	)
-	(wire
-		(pts
 			(xy 209.55 115.57) (xy 209.55 118.11)
 		)
@@
 	(wire
 		(pts
+			(xy 224.79 29.21) (xy 224.79 33.02)
+		)
+		(stroke
+			(width 0)
+			(type default)
+		)
+	)
+	(wire
+		(pts
 			(xy 218.44 24.13) (xy 213.36 24.13)
 		)
@@
 					(unit 1)
 				)
-			)
-		)
-	)
-	(symbol
-		(lib_name "SolderJumper_3_Open_1")
-		(lib_id "Jumper:SolderJumper_3_Open")
-		(at 227.33 33.02 180)
-		(unit 1)
-		(exclude_from_sim no)
-		(in_bom no)
-		(on_board yes)
-		(dnp no)
-		(property "Reference" "JP1"
-			(at 229.616 30.734 0)
-			(effects
-				(font
-					(size 1.27 1.27)
-				)
-			)
-		)
-		(property "Value" "BypassBattery"
-			(at 229.362 35.306 0)
-			(effects
-				(font
-					(size 1.27 1.27)
-				)
-			)
-		)
-		(property "Footprint" "Jumper:SolderJumper-3_P1.3mm_Open_RoundedPad1.0x1.5mm_NumberLabels"
-			(at 227.33 33.02 0)
-			(effects
-				(font
-					(size 1.27 1.27)
-				)
-				(hide yes)
-			)
-		)
-		(property "Datasheet" "~"
-			(at 227.33 33.02 0)
-			(effects
-				(font
-					(size 1.27 1.27)
-				)
-				(hide yes)
-			)
-		)
-		(property "Description" "Solder Jumper, 3-pole, open"
-			(at 227.33 33.02 0)
-			(effects
-				(font
-					(size 1.27 1.27)
-				)
-				(hide yes)
-			)
-		)
-		(pin "3"
-		)
-		(pin "2"
-		)
-		(pin "1"
-		)
-		(instances
-			(project ""
-				(path "/eee23683-93c4-45fa-9c00-e358d0d25f58"
-					(reference "JP1")
-					(unit 1)
-				)
